File: bartlepslit.kicad_pcb (KiCad board)
At the start: 2 copper layers, 336.7 x 119.6 mm, 119 parts, among them K1 SW_Push, K10 SW_Push, K11 SW_Push, K12 SW_Push, K13 SW_Push, K14 SW_Push, K15 SW_Push, K16 SW_Push, K17 SW_Push, K18 SW_Push, K19 SW_Push, K2 SW_Push, K20 SW_Push, K21 SW_Push, K22 SW_Push, K23 SW_Push, K24 SW_Push, K25 SW_Push, K26 SW_Push, K27 SW_Push, K28 SW_Push, K29 SW_Push, K3 SW_Push, K30 SW_Push, K31 SW_Push, K32 SW_Push, K33 SW_Push, K34 SW_Push, K35 SW_Push, K36 SW_Push, K37 SW_Push, K38 SW_Push, K39 SW_Push, K4 SW_Push, K40 SW_Push, K41 SW_Push, K42 SW_Push, K5 SW_Push, K6 SW_Push, K7 SW_Push, K8 SW_Push, K9 SW_Push, U1 ProMicro

Commit message: feat: optimized break off parts
Parts:
- moved REF** 23.2 mm to (125.8, 129.4), turned to 180 degrees
- moved REF** 22.9 mm to (276.4, 129.2), turned to 0 degrees
- moved REF** 21.0 mm to (108.3, 129.4), turned to 180 degrees
- moved REF** 20.9 mm to (293.9, 129.2), turned to 0 degrees
Other:
- outline, holes or cut-outs redrawn

Commit message: feat: added missing reset switch
Parts:
- added SW1: SW_Push, Button_Switch_SMD:SW_Tactile_SPST_NO_Straight_CK_PTS636Sx25SMTRLFS, B.Cu at (194.8, 67.3)
Connections:
- net Net-(U1-RST) renamed RST
Routing:
- net RST: track 15.5 -> 19.3 mm
- net GND: track 15.5 -> 19.3 mm
